Commit message: fix(quad): 02_Leg hip/thigh inertial 좌우 대칭화(평균) + walk_loop MAXITER/NWARM env
- URDF/MJCF의 hip(117g/COM19mm)·thigh(미세) 좌우 비대칭(CAD 미러 오류 추정)을
  평균+미러규칙으로 대칭화(총질량 보존). MuJoCo fullinertia 사용. 모델 좌우 완벽대칭.
  ※단 이 비대칭은 측방 쏠림(limp)의 원인 아님으로 확인됨(대칭화 후도 −10cm 동일).
   limp/측방오프셋의 실제 원인은 pin↔MuJoCo 실행 불일치(제어측).
- walk_loop에 MAXITER/NWARM env(고속 계획수렴 튜닝용).

고속 보행 탐색: 고정사이클 walk_loop은 측방 Floquet 불안정으로 ~0.4m/s가 한계
(튜닝 max ~10s). 돌파엔 capture-point/RTI/WBC 등 구조변경 필요(사용자: 보류).

Co-Authored-By: Claude Opus 4.8 <noreply@anthropic.com>

File: quad/urdf/02_Leg_UFDF_260610_8.urdf (robot description, URDF)
Before this commit: robot 02_Leg_UFDF_260610_8, 21 links, 20 joints
Links:
- link FL_hip_link: mass 1.385 -> 1.3265
- link FR_hip_link: mass 1.268 -> 1.3265
- link HL_hip_link: mass 1.268 -> 1.3265
- link HR_hip_link: mass 1.385 -> 1.3265
